File: mjspcb.sch (KiCad schematic (older format))
At the start: 34 parts, among them P1 2.7 - 6.0 VDC, P2 serial breakout, P3 HTU21D breakout, P4 GPS, P5 piezo, P6 BPW34, P7 electrodes, P8 perfboard breakout, Q1 STU60N3LH5, Q2 STU60N3LH5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

Commit message: Revision 2 of Meet je stad PCB
*added reset header
*changed pinout of I2C breakout to accomodate Sparkfun Si7021
*various minor other modifications
Parts:
- added JP2: V1, meetjestad:SOLDER-JUMPER_2-WAY-CLOSED, symbol JUMPER_3-PIN-CLOSED
- added JP3: V2, meetjestad:SOLDER-JUMPER_2-WAY-CLOSED, symbol JUMPER_3-PIN-CLOSED
- added P9: reset, Socket_Strips:Socket_Strip_Straight_1x02, symbol CONN_01X02
- C2: value 10u -> 100u
- D1: symbol LED -> LED-RESCUE-mjspcb
- P3: value HTU21D breakout -> I2C breakout
- Q1: symbol FDP7030BL -> STU60N3LH5
Connections:
- wire segments 132 -> 138
Other:
- note added: "www.sparkfun.com/products/13763"
- note removed: "www.sparkfun.com/products/12064"
- moved on the sheet: P2, P3, P4, P5, P6, P7, R10, R11, R12, R13, R8, R9

Commit message: Convert schematic to KiCad 5
In KiCad 5, symbols reference the library they are in explicitly. Also,
a lot of symbols were changed for more consistency. This commit changes
all symbols to their new version in the official libraries, removing the
need for our own symbol library (which is removed by this commit).

For the STU MOSFET component, not specific symbol is available, so a
generic MOSFET symbol is used instead.

This also updates the footprint fields to point to versions from the
KiCad 5 libraries, but does not update the actual layout to use them
yet.

For the GPS connector symbol, the pinout was reversed (matching the,
technically incorrect, footprint used). This fixes the pin order in the
schematic and updates the footprint field to a footprint that matches
this pin order, so when a netlist is imported in the future, this should
still match.
Parts:
- removed U2: RFM95W, meetjestad:RFM95W, symbol RFM95W
- added U2: RFM95W, RF_Module:HOPERF_RFM9XW_SMD, symbol RF_AM_FM:RFM95W-868S2
- AE1: footprint Pin_Headers:Pin_Header_Straight_1x01 -> Connector_PinHeader_2.54mm:PinHeader_1x01_P2.54mm_Vertical; symbol Antenna_Helical -> Device:Antenna
- C1, C3, C5: footprint Capacitors_ThroughHole:C_Disc_D3_P2.5 -> Capacitor_THT:C_Disc_D3.0mm_W1.6mm_P2.50mm; symbol C -> Device:C
- C2, C4: footprint Capacitors_ThroughHole:C_Radial_D5_L11_P2 -> Capacitor_THT:CP_Radial_D5.0mm_P2.00mm; symbol CP -> Device:CP
- D1: footprint LEDs:LED-3MM -> LED_THT:LED_D3.0mm; symbol LED-RESCUE-mjspcb -> Device:LED
- JP1: footprint Pin_Headers:Pin_Header_Straight_1x03 -> Connector_PinHeader_2.54mm:PinHeader_1x03_P2.54mm_Vertical; symbol JUMPER3 -> Jumper:Jumper_3_Open
- JP2, JP3: footprint meetjestad:SOLDER-JUMPER_2-WAY-CLOSED -> Jumper:SolderJumper-3_P1.3mm_Bridged12_Pad1.0x1.5mm; symbol JUMPER_3-PIN-CLOSED -> Jumper:SolderJumper_3_Bridged12
- P1: footprint meetjestad:Batterypack3xAAA -> Battery:BatteryHolder_Keystone_2479_3xAAA; symbol CONN_01X02 -> Connector_Generic:Conn_01x02
- P2: footprint Pin_Headers:Pin_Header_Straight_1x06 -> Connector_PinHeader_2.54mm:PinHeader_1x06_P2.54mm_Vertical; symbol CONN_01X06 -> Connector_Generic:Conn_01x06
- P3: footprint Socket_Strips:Socket_Strip_Straight_1x04 -> Connector_PinSocket_2.54mm:PinSocket_1x04_P2.54mm_Vertical; symbol CONN_01X04 -> Connector_Generic:Conn_01x04
- P4: footprint Pin_Headers:Pin_Header_Angled_1x03 -> Connector_JST:JST_PH_S3B-PH-K_1x03_P2.00mm_Horizontal; symbol CONN_01X03 -> Connector_Generic:Conn_01x03
- P5, P6, P7, P9: footprint Socket_Strips:Socket_Strip_Straight_1x02 -> Connector_PinHeader_2.54mm:PinHeader_1x02_P2.54mm_Vertical; symbol CONN_01X02 -> Connector_Generic:Conn_01x02
- P8: footprint meetjestad:Perf_board_connecttion_1x11 -> Connector_PinHeader_2.54mm:PinHeader_1x11_P2.54mm_Vertical; symbol CONN_01X11 -> Connector_Generic:Conn_01x11
- Q1, Q2: footprint TO-251 -> Package_TO_SOT_THT:TO-251-3_Vertical; symbol STU60N3LH5 -> Device:Q_NMOS_GDS
- R1, R10, R11, R12, R13, R2, R3, R4, R5, R6, R7, R8, R9: footprint Resistors_ThroughHole:Resistor_Horizontal_RM10mm -> Resistor_THT:R_Axial_DIN0207_L6.3mm_D2.5mm_P10.16mm_Horizontal; symbol R -> Device:R
- U1: footprint DIP-28 -> Package_DIP:DIP-28_W7.62mm_Socket; symbol ATMEGA328-P -> MCU_Microchip_ATmega:ATmega328P-PU
- U3: footprint TO-92 -> Package_TO_SOT_THT:TO-92_Inline; symbol MCP1700-2502E/TO -> Regulator_Linear:MCP1700-3302E_TO92
Connections:
- net GND: now also JP2.3 (B), U2.1 (GND), U2.10 (GND), U2.8 (GND); no longer JP2.2
- net VCC: now also JP3.3 (B), P4.3 (Pin_3), U2.13 (3.3V); no longer JP3.2, P4.1 (P1)
- net D9: now reaches U1.15 (PB1)
- net D9: now also U2.6 (RESET)
- net D10: now reaches R2.2, U1.16 (PB2)
- net D10: now also U2.5 (NSS)
- net MOSI: now reaches U1.17 (PB3)
- net MOSI: now also U2.3 (MOSI)
- net MISO: now reaches U1.18 (PB4)
- net MISO: now also U2.2 (MISO)
- net SCK: now reaches U1.19 (PB5)
- net SCK: now also U2.4 (SCK)
- net D2: now reaches U1.4 (PD2)
- net D2: now also U2.14 (DIO0)
- net D3: now reaches U1.5 (PD3)
- net D3: now also U2.15 (DIO1)
- net D4: now reaches U1.6 (PD4)
- net D4: now also U2.16 (DIO2)
- net at AE1.1 (A): now also U2.9 (ANT)
- net at P3.1 (Pin_1): now also JP3.2 (C); no longer JP3.1
- net at P3.2 (Pin_2): now also JP2.2 (C); no longer JP2.1
- net at R8.1: now also P4.1 (Pin_1); no longer P4.3 (P3)
- no-connect marks 0 -> 4
Other:
- moved on the sheet: AE1, C1, R1, R2, R4
